Commit message: fix:缩小叉车模型,修复联合训练bobot2规划失败的bug,修改forklift的costmap

File: src/sim_env/urdf/forklift/forklift.gazebo.xacro (robot description, xacro)
@@ -101,5 +101,5 @@
         </scan>
         <range>
-          <min>0.45</min>
+          <min>0.17</min>
           <max>100</max>
           <resolution>0.015</resolution>
@@ -183,6 +183,6 @@
       <leftRearJoint>rear_left_wheel_joint</leftRearJoint>
       <rightRearJoint>rear_right_wheel_joint</rightRearJoint>
-      <wheelSeparation>0.36</wheelSeparation> <!-- 左右轮距离 -->
-      <wheelDiameter>0.18</wheelDiameter>   <!-- 轮子直径 -->
+      <wheelSeparation>0.12</wheelSeparation> <!-- 左右轮距离 缩放为原来的1/3 -->
+      <wheelDiameter>0.06</wheelDiameter>   <!-- 轮子直径 缩放为原来的1/3 -->
       <torque>500</torque>                 <!-- 扭矩 -->
       <commandTopic>cmd_vel</commandTopic>

File: src/sim_env/urdf/forklift/forklift.urdf.xacro (robot description, xacro)
@@ -3,16 +3,16 @@
   <xacro:include filename="$(find sim_env)/urdf/forklift/forklift_base.xacro" />
   <!-- Camera property definitions (keep from original model) -->
-  <xacro:property name="r200_cam_rgb_px" value="0.005" />
-  <xacro:property name="r200_cam_rgb_py" value="0.018" />
-  <xacro:property name="r200_cam_rgb_pz" value="0.013" />
-  <xacro:property name="r200_cam_depth_offset" value="0.01" />
+  <xacro:property name="r200_cam_rgb_px" value="0.0017" />
+  <xacro:property name="r200_cam_rgb_py" value="0.006" />
+  <xacro:property name="r200_cam_rgb_pz" value="0.0043" />
+  <xacro:property name="r200_cam_depth_offset" value="0.0033" />
   <!-- Base footprint as root - 必须有惯性参数才能让 Gazebo 正确计算速度 -->
   <link name="base_footprint">
     <inertial>
-      <mass value="0.0001"/>
+      <mass value="0.0000037"/>
       <origin xyz="0 0 0"/>
-      <inertia ixx="0.0001" ixy="0" ixz="0"
-              iyy="0.0001" iyz="0"
-              izz="0.0001"/>
+      <inertia ixx="0.0000037" ixy="0" ixz="0"
+              iyy="0.0000037" iyz="0"
+              izz="0.0000037"/>
     </inertial>
   </link>
@@ -23,13 +23,13 @@
     <parent link="front_axle" />
     <child link="imu_link" />
-    <origin xyz="0.0 0 0.068" rpy="0 0 0" />
+    <origin xyz="0.0 0 0.0227" rpy="0 0 0" />
   </joint>
   <link name="imu_link">
     <inertial>
-      <mass value="0.001"/>
+      <mass value="0.000037"/>
       <origin xyz="0 0 0"/>
-      <inertia ixx="0.0001" ixy="0" ixz="0"
-              iyy="0.0001" iyz="0"
-              izz="0.0001"/>
+      <inertia ixx="0.0000037" ixy="0" ixz="0"
+              iyy="0.0000037" iyz="0"
+              izz="0.0000037"/>
     </inertial>
   </link>
@@ -38,5 +38,5 @@
     <parent link="front_axle" />
     <child link="base_scan" />
-    <origin xyz="-0.35 0 0.65" rpy="0 0 0" />
+    <origin xyz="-0.1167 0 0.0833" rpy="0 0 0" />
   </joint>
   <link name="base_scan">
@@ -44,25 +44,25 @@
       <origin xyz="0 0 0" rpy="0 0 0" />
       <geometry>
-        <mesh filename="package://sim_env/meshes/turtlebot3/sensors/lds.stl" scale="0.001 0.001 0.001" />
+        <mesh filename="package://sim_env/meshes/turtlebot3/sensors/lds.stl" scale="0.000333 0.000333 0.000333" />
       </geometry>
       <material name="dark" />
     </visual>
     <collision>
-      <origin xyz="0.015 0 -0.0065" rpy="0 0 0" />
+      <origin xyz="0.005 0 -0.0022" rpy="0 0 0" />
       <geometry>
-        <cylinder length="0.0315" radius="0.055" />
+        <cylinder length="0.0105" radius="0.0183" />
       </geometry>
     </collision>
     <inertial>
-      <mass value="0.114" />
+      <mass value="0.0042" />
       <origin xyz="0 0 0" />
-      <inertia ixx="0.001" ixy="0.0" ixz="0.0"
-               iyy="0.001" iyz="0.0"
-               izz="0.001" />
+      <inertia ixx="0.000037" ixy="0.0" ixz="0.0"
+               iyy="0.000037" iyz="0.0"
+               izz="0.000037" />
     </inertial>
   </link>
   <!-- Realsense camera on chassis -->
   <joint name="camera_joint" type="fixed">
-    <origin xyz="0.064 -0.065 0.5" rpy="0 0 0" />
+    <origin xyz="0.0213 -0.0217 0.1667" rpy="0 0 0" />
     <parent link="front_axle" />
     <child link="camera_link" />
@@ -76,7 +76,7 @@
     </visual>
     <collision>
-      <origin xyz="0.003 0.065 0.007" rpy="0 0 0" />
+      <origin xyz="0.001 0.0217 0.0023" rpy="0 0 0" />
       <geometry>
-        <box size="0.012 0.132 0.020" />
+        <box size="0.004 0.044 0.0067" />
       </geometry>
     </collision>

File: src/sim_env/urdf/forklift/forklift_base.xacro (robot description, xacro)
@@ -2,5 +2,5 @@
 <robot xmlns:xacro="http://ros.org/wiki/xacro">
   <!-- 定义参数 用于轮子的尺寸和缩放比例 -->
-  <xacro:property name="wheel_mesh_scale" value="0.3"/>
+  <xacro:property name="wheel_mesh_scale" value="0.1"/>
   <xacro:property name="wheel_radius_origin" value="0.3"/>
   <xacro:property name="wheel_length_origin" value="0.2"/>
@@ -33,5 +33,5 @@
     <link name="front_axle">
       <visual>
-        <origin xyz="-0.3 0 0.22" rpy="0 0 0"/>
+        <origin xyz="-0.1 0 0.0733" rpy="0 0 0"/>
         <geometry>
           <mesh filename="package://sim_env/meshes/fork/forklift_base2.dae" scale="${wheel_mesh_scale} ${wheel_mesh_scale} ${wheel_mesh_scale}"/>
@@ -39,10 +39,10 @@
       </visual>
       <collision>
-        <origin xyz="-0.3 0 0.22" rpy="0 0 0"/>
+        <origin xyz="-0.1 0 0.0733" rpy="0 0 0"/>
         <geometry>
-          <box size="0.6 0.4 0.3"/>
+          <box size="0.2667 0.1333 0.1"/>
         </geometry>
       </collision>
-      <xacro:box_inertial x="0.6" y="0.4" z="0.3" mass="0.5" />
+      <xacro:box_inertial x="0.2667" y="0.1333" z="0.1" mass="0.0185" />
     </link>
     <joint name="front_joint_odom" type="fixed">
@@ -67,11 +67,11 @@
       </collision>
       <xacro:cylinder_inertial radius="${wheel_radius_origin * wheel_mesh_scale}"
-                                length="${wheel_length_origin * wheel_mesh_scale}"
-                                mass="0.75" />
+                length="${wheel_length_origin * wheel_mesh_scale}"
+                mass="0.0278" />
     </link>
     <joint name="rear_left_wheel_joint" type="continuous">
       <parent link="front_axle"/>
       <child  link="rear_left_wheel_link"/>
-      <origin xyz="-0.6 0.18 0.08" rpy="0 0 0"/>
+      <origin xyz="-0.2 0.06 0.0267" rpy="0 0 0"/>
       <axis xyz="0 1 0"/>
     </joint>
@@ -92,11 +92,11 @@
       </collision>
       <xacro:cylinder_inertial radius="${wheel_radius_origin * wheel_mesh_scale}"
-                                length="${wheel_length_origin * wheel_mesh_scale}"
-                                mass="0.75" />
+                length="${wheel_length_origin * wheel_mesh_scale}"
+                mass="0.0278" />
     </link>
     <joint name="rear_right_wheel_joint" type="continuous">
       <parent link="front_axle"/>
       <child link="rear_right_wheel_link"/>
-      <origin xyz="-0.6 -0.18 0.08" rpy="0 0 0"/>
+      <origin xyz="-0.2 -0.06 0.0267" rpy="0 0 0"/>
       <axis xyz="0 1 0"/>
     </joint>
@@ -117,11 +117,11 @@
       </collision>
       <xacro:cylinder_inertial radius="${wheel_radius_origin * wheel_mesh_scale}"
-                                length="${wheel_length_origin * wheel_mesh_scale}"
-                                mass="0.5" />
+                length="${wheel_length_origin * wheel_mesh_scale}"
+                mass="0.0185" />
     </link>
     <joint name="front_left_wheel_joint" type="continuous">
       <parent link="front_axle"/>
       <child link="front_left_wheel_link"/>
-      <origin xyz="-0.10 0.18 0.08" rpy="0 0 0"/>
+      <origin xyz="-0.0333 0.06 0.0267" rpy="0 0 0"/>
       <axis xyz="0 1 0"/>
     </joint>
@@ -142,11 +142,11 @@
       </collision>
       <xacro:cylinder_inertial radius="${wheel_radius_origin * wheel_mesh_scale}"
-                                length="${wheel_length_origin * wheel_mesh_scale}"
-                                mass="0.5" />
+                length="${wheel_length_origin * wheel_mesh_scale}"
+                mass="0.0185" />
     </link>
     <joint name="front_right_wheel_joint" type="continuous">
       <parent link="front_axle"/>
       <child link="front_right_wheel_link"/>
-      <origin xyz="-0.10 -0.18 0.08" rpy="0 0 0"/>
+      <origin xyz="-0.0333 -0.06 0.0267" rpy="0 0 0"/>
       <axis xyz="0 1 0"/>
     </joint>
