Commit message: fix:修复pioneer3dx激光雷达检测不到forklift

File: src/sim_env/urdf/forklift/forklift.urdf.xacro (robot description, xacro)
@@ -62,4 +62,25 @@
     </inertial>
   </link>
+  <!-- Additional collision element for laser detection -->
+  <joint name="laser_detection_joint" type="fixed">
+    <parent link="front_axle" />
+    <child link="laser_detection_element" />
+    <origin xyz="0 0 0.25" rpy="0 0 0" />
+  </joint>
+  <link name="laser_detection_element">
+    <collision>
+      <origin xyz="0 0 0" rpy="0 0 0" />
+      <geometry>
+        <box size="0.3 0.2 0.1" />
+      </geometry>
+    </collision>
+    <inertial>
+      <mass value="0.001" />
+      <origin xyz="0 0 0" />
+      <inertia ixx="0.000001" ixy="0.0" ixz="0.0"
+               iyy="0.000001" iyz="0.0"
+               izz="0.000001" />
+    </inertial>
+  </link>
   <!-- Realsense camera on chassis -->
   <joint name="camera_joint" type="fixed">

Commit message: feat: add clamp plates to forklift model

File: src/sim_env/urdf/forklift/forklift.urdf.xacro (robot description, xacro)
@@ -127,3 +127,38 @@
   </joint>
   <link name="camera_depth_optical_frame" />
+  <!-- Two clamp plates at the front of the forklift -->
+  <!-- Left clamp plate -->
+  <link name="left_clamp_plate">
+    <visual>
+      <origin xyz="0 0 0" rpy="0 0 0"/>
+      <geometry>
+        <box size="0.15 0.005 0.08"/>
+      </geometry>
+      <material name="gray">
+        <color rgba="0.5 0.5 0.5 1.0"/>
+      </material>
+    </visual>
+  </link>
+  <joint name="left_clamp_joint" type="fixed">
+    <parent link="front_axle"/>
+    <child link="left_clamp_plate"/>
+    <origin xyz="0.08 0.04 0.05" rpy="0 0 0"/>
+  </joint>
+  <!-- Right clamp plate -->
+  <link name="right_clamp_plate">
+    <visual>
+      <origin xyz="0 0 0" rpy="0 0 0"/>
+      <geometry>
+        <box size="0.15 0.005 0.08"/>
+      </geometry>
+      <material name="gray">
+        <color rgba="0.5 0.5 0.5 1.0"/>
+      </material>
+    </visual>
+  </link>
+  <joint name="right_clamp_joint" type="fixed">
+    <parent link="front_axle"/>
+    <child link="right_clamp_plate"/>
+    <origin xyz="0.08 -0.04 0.05" rpy="0 0 0"/>
+  </joint>
 </robot>
